Commit message: LIVO

File: linorobot2/linorobot2_description/urdf/mecanum_properties.urdf.xacro (robot description, xacro)
@@ -22,9 +22,9 @@
 <!--depthcam-->
   <xacro:property name="depth_sensor_pose">
-    <origin xyz="0.204 0 0.6" rpy="0 0.523599 0"/>
+    <origin xyz="0.204 0 0.6" rpy="0 0 0"/>
   </xacro:property>
 <!--imu-->
   <xacro:property name="depth_sensor_pose">
-    <origin xyz="0.204 0 0.6" rpy="0 0.523599 0"/>
+    <origin xyz="0.204 0 0.6" rpy="0 0 0"/>
   </xacro:property>
 </robot>

File: linorobot2/linorobot2_description/urdf/sensors/depth_sensor.urdf.xacro (robot description, xacro)
@@ -38,5 +38,5 @@
     </gazebo>rgb(213,28,40)
     <joint name="camera_to_base_link" type="fixed">
-      <origin xyz="0.204 0 0.6" rpy="0 0.523599 0"/>
+      <origin xyz="0.204 0 0.6" rpy="0 0 0"/>
       <parent link="base_link"/>
       <child link="camera_link"/>
